File: KiCAD/TRS80_Model_I_Keyboard_MX_Full_E2.kicad_pcb (KiCad board)
At the start: 2 copper layers, 375 x 94.5 mm, 92 parts, among them J1 Connection Keyboad Side, J10 Reset, SW1 @, SW10 A, SW11 I, SW12 Q, SW13 Y, SW14 1, SW15 9, SW16 CLEAR, SW17 B, SW18 J, SW19 R, SW2 H, SW20 Z, SW21 2, SW22 :, SW23 BREAK, SW24 C, SW25 K, SW26 S, SW27 3, SW28 ;, SW29 UP, SW3 P, SW30 D, SW31 L, SW32 T, SW33 4, SW34 ,, SW35 DOWN, SW36 E, SW37 M, SW38 U, SW39 5, SW4 X, SW40 -, SW41 LEFT, SW42 F, SW43 N, SW44 V, SW45 6, SW46 ., SW47 RIGHT, SW48 G, SW49 O, SW5 0, SW50 W, SW51 7, SW52 /, SW53 SPACE, SW54 0, SW55 8, SW56 ENTER, SW57 1, SW58 9, SW59 2, SW6 8, SW60 3, SW61 4, SW62 5, SW63 6, SW64 ., SW65 7, SW66 SPACE, SW67 X1, SW68 X2, SW69 SPACE, SW7 ENTER, SW70 SW_DIP_x09, SW71 SW_DIP_x09, SW72 SW_DIP_x09, SW73 SW_DIP_x09, SW74 SW_DIP_x09, SW75 SW_DIP_x09, SW76 SW_DIP_x09, SW77 SW_DIP_x09, SW8 LSHIFT, SW9 RSHIFT

Commit message: E2E changes
Parts:
- SW53, SW66: footprint Button_Switch_Keyboard:SW_Cherry_MX_1.00u_PCB -> RetroStackLibrary:SW_Cherry_MX_1.00u_PCB_Spacebar_Universal
- moved SW53 5.83 mm to (106.3, 86.7)
- moved SW66 5.25 mm to (202.7, 86.7)
Routing:
- net /A0: track 91.4 -> 95.4 mm
- net R7: track 592.0 -> 594.7 mm
- net GND: track 456.8 -> 458.9 mm
- net R5: track 660.7 -> 662.3 mm
- net C2: track 684.7 -> 686.1 mm
- net R6: track 673.3 -> 674.1 mm
- net /D1: track 41.0 -> 41.6 mm
- net Net-(SW68-Pad1): track 59.5 -> 60.1 mm
Other:
- board text added: "MX Keyboard"
- board text added: "TRS-80 Model 1"
- board text removed: "TRS-80 Model 1 MX Keyboard"

Commit message: E2F version
Routing:
- net /A7: track 62.7 -> 70.1 mm
- net /A3: track 71.9 -> 78.8 mm
- net R7: track 594.7 -> 601.5 mm
- net /A1: track 72.3 -> 78.8 mm
- net /A6: track 71.5 -> 77.4 mm
- net R3: track 529.8 -> 534.9 mm
- net /A5: track 83.5 -> 88.4 mm
- net /A2: track 69.0 -> 73.4 mm
- net C6: track 670.6 -> 674.9 mm
- net C5: track 566.5 -> 569.9 mm
- net C4: track 625.0 -> 628.2 mm
- net +5V: track 379.9 -> 382.3 mm
- net GND: track 458.9 -> 461.3 mm
- net R1: track 511.4 -> 513.5 mm
- net /A4: track 83.0 -> 84.9 mm
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Other:
- outline, holes or cut-outs redrawn
- board text added: "E2F"
- board text removed: "E2E"
