File: KiCAD/TRS80_Model_I_Keyboard_MX_Full_E2.kicad_sch (KiCad schematic)
At the start: 76 parts, among them J1 Connection Keyboad Side, J10 Reset, SW1 @, SW10 A, SW11 I, SW12 Q, SW13 Y, SW14 1, SW15 9, SW17 B, SW18 J, SW19 R, SW2 H, SW20 Z, SW21 2, SW22 :, SW24 C, SW25 K, SW26 S, SW27 3, SW28 ;, SW29 UP, SW3 P, SW30 D, SW31 L, SW32 T, SW33 4, SW34 ,, SW35 DOWN, SW36 E, SW37 M, SW38 U, SW39 5, SW4 X, SW40 -, SW41 LEFT, SW42 F, SW43 N, SW44 V, SW45 6, SW46 ., SW47 RIGHT, SW48 G, SW49 O, SW5 0, SW50 W, SW51 7, SW52 /, SW53 SPACE, SW54 0, SW55 8, SW56 ENTER, SW57 1, SW58 9, SW59 2, SW6 8, SW60 3, SW61 4, SW62 5, SW63 6, SW64 ., SW65 7, SW66 SPACE, SW69 SPACE, SW7 ENTER, SW8 LSHIFT, SW9 RSHIFT

Commit message: E2E changes
Parts:
- SW53, SW66: footprint Button_Switch_Keyboard:SW_Cherry_MX_1.00u_PCB -> RetroStackLibrary:SW_Cherry_MX_1.00u_PCB_Spacebar_Universal
Other:
- moved on the sheet: SW53, SW66, SW69
Changed lines of the file:
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@@
   (title_block
     (title "TRS-80 Model I - MX Keyboard Full")
-    (date "2024-04-13")
+    (date "2024-05-17")
     (rev "E2E")
     (company "RetroStack - Marcel Erz")
@@
   (junction (at 220.98 59.69) (diameter 0) (color 0 0 0 0)
   )
-  (junction (at 245.11 101.6) (diameter 0) (color 0 0 0 0)
-  )
   (junction (at 196.85 102.87) (diameter 0) (color 0 0 0 0)
   )
@@
   (junction (at 243.205 101.6) (diameter 0) (color 0 0 0 0)
   )
+  (junction (at 255.27 99.06) (diameter 0) (color 0 0 0 0)
+  )
   (junction (at 231.14 20.955) (diameter 0) (color 0 0 0 0)
   )
@@
   (junction (at 184.785 59.69) (diameter 0) (color 0 0 0 0)
   )
-  (junction (at 255.27 97.155) (diameter 0) (color 0 0 0 0)
-  )
   (junction (at 160.655 80.01) (diameter 0) (color 0 0 0 0)
   )
@@
   (junction (at 208.915 81.28) (diameter 0) (color 0 0 0 0)
   )
+  (junction (at 255.27 106.68) (diameter 0) (color 0 0 0 0)
+  )
   (junction (at 233.045 80.01) (diameter 0) (color 0 0 0 0)
   )
@@
   (junction (at 118.11 195.58) (diameter 0) (color 0 0 0 0)
   )
-  (junction (at 255.27 101.6) (diameter 0) (color 0 0 0 0)
-  )
   (junction (at 160.655 102.87) (diameter 0) (color 0 0 0 0)
   )
@@
   (junction (at 170.815 90.805) (diameter 0) (color 0 0 0 0)
   )
+  (junction (at 255.27 102.87) (diameter 0) (color 0 0 0 0)
+  )
   (junction (at 182.88 58.42) (diameter 0) (color 0 0 0 0)
   )
@@
   (junction (at 194.945 75.565) (diameter 0) (color 0 0 0 0)
   )
-  (junction (at 255.27 106.045) (diameter 0) (color 0 0 0 0)
-  )
   (junction (at 170.815 80.01) (diameter 0) (color 0 0 0 0)
   )
@@
     (stroke (width 0) (type default))
   )
-  (wire (pts (xy 89.535 69.215) (xy 89.535 140.335))
+  (wire (pts (xy 255.27 106.68) (xy 255.27 117.475))
     (stroke (width 0) (type default))
   )
-  (wire (pts (xy 245.11 97.155) (xy 245.11 101.6))
+  (wire (pts (xy 89.535 69.215) (xy 89.535 140.335))
     (stroke (width 0) (type default))
   )
@@
     (stroke (width 0) (type default))
   )
-  (wire (pts (xy 255.27 97.155) (xy 255.27 101.6))
+  (wire (pts (xy 255.27 90.805) (xy 255.27 99.06))
     (stroke (width 0) (type default))
   )
@@
     (stroke (width 0) (type default))
   )
-  (wire (pts (xy 255.27 106.045) (xy 255.27 117.475))
-    (stroke (width 0) (type default))
-  )
   (wire (pts (xy 99.06 185.42) (xy 99.06 195.58))
     (stroke (width 0) (type default))
@@
     (stroke (width 0) (type default))
   )
-  (wire (pts (xy 245.11 102.87) (xy 245.11 106.045))
+  (wire (pts (xy 245.11 102.87) (xy 245.11 106.68))
     (stroke (width 0) (type default))
   )
@@
     (stroke (width 0) (type default))
   )
+  (wire (pts (xy 255.27 99.06) (xy 255.27 102.87))
+    (stroke (width 0) (type default))
+  )
   (wire (pts (xy 170.815 75.565) (xy 170.815 80.01))
     (stroke (width 0) (type default))
@@
     (stroke (width 0) (type default))
   )
-  (wire (pts (xy 255.27 101.6) (xy 255.27 106.045))
-    (stroke (width 0) (type default))
-  )
   (wire (pts (xy 233.045 90.805) (xy 233.045 92.075))
     (stroke (width 0) (type default))
@@
     (stroke (width 0) (type default))
   )
+  (wire (pts (xy 255.27 102.87) (xy 255.27 106.68))
+    (stroke (width 0) (type default))
+  )
   (wire (pts (xy 243.205 86.36) (xy 243.205 90.805))
     (stroke (width 0) (type default))
@@
     (stroke (width 0) (type default))
   )
-  (wire (pts (xy 255.27 90.805) (xy 255.27 97.155))
-    (stroke (width 0) (type default))
-  )
   (wire (pts (xy 207.01 142.875) (xy 207.01 132.715))
     (stroke (width 0) (type default))
@@
     (stroke (width 0) (type default))
   )
-  (wire (pts (xy 245.11 102.87) (xy 245.11 101.6))
-    (stroke (width 0) (type default))
-  )
   (wire (pts (xy 62.23 140.335) (xy 62.23 139.065))
     (stroke (width 0) (type default))
@@
     (stroke (width 0) (type default))
   )
+  (wire (pts (xy 245.11 99.06) (xy 245.11 102.87))
+    (stroke (width 0) (type default))
+  )
   (wire (pts (xy 170.815 58.42) (xy 170.815 69.215))
     (stroke (width 0) (type default))
@@
     )
   )
-  (symbol (lib_id "Switch:SW_Push") (at 250.19 97.155 0) (mirror y) (unit 1)
+  (symbol (lib_id "Switch:SW_Push") (at 250.19 99.06 0) (mirror y) (unit 1)
     (in_bom yes) (on_board yes) (dnp no)
-    (property "Reference" "SW66" (at 254 95.25 0)
+    (property "Reference" "SW66" (at 254 97.155 0)
       (effects (font (size 0.8 0.8)) (justify left))
     )
-    (property "Value" "SPACE" (at 250.19 97.155 0)
+    (property "Value" "SPACE" (at 250.19 99.06 0)
       (effects (font (size 0.6 0.6)))
     )
-    (property "Footprint" "Button_Switch_Keyboard:SW_Cherry_MX_1.00u_PCB" (at 250.19 92.075 0)
+    (property "Footprint" "RetroStackLibrary:SW_Cherry_MX_1.00u_PCB_Spacebar_Universal" (at 250.19 93.98 0)
       (effects (font (size 1.27 1.27)) hide)
     )
-    (property "Datasheet" "~" (at 250.19 92.075 0)
+    (property "Datasheet" "~" (at 250.19 93.98 0)
       (effects (font (size 1.27 1.27)) hide)
     )
@@
     )
   )
-  (symbol (lib_id "Switch:SW_Push") (at 250.19 106.045 0) (mirror y) (unit 1)
+  (symbol (lib_id "Switch:SW_Push") (at 250.19 106.68 0) (mirror y) (unit 1)
     (in_bom yes) (on_board yes) (dnp no)
-    (property "Reference" "SW69" (at 254 104.14 0)
+    (property "Reference" "SW69" (at 254 104.775 0)
       (effects (font (size 0.8 0.8)) (justify left))
     )
-    (property "Value" "SPACE" (at 250.19 106.045 0)
+    (property "Value" "SPACE" (at 250.19 106.68 0)
       (effects (font (size 0.6 0.6)))
     )
-    (property "Footprint" "Button_Switch_Keyboard:SW_Cherry_MX_1.00u_PCB" (at 250.19 100.965 0)
+    (property "Footprint" "Button_Switch_Keyboard:SW_Cherry_MX_1.00u_PCB" (at 250.19 101.6 0)
       (effects (font (size 1.27 1.27)) hide)
     )
-    (property "Datasheet" "~" (at 250.19 100.965 0)
+    (property "Datasheet" "~" (at 250.19 101.6 0)
       (effects (font (size 1.27 1.27)) hide)
     )
@@
     )
   )
-  (symbol (lib_id "Switch:SW_Push") (at 250.19 101.6 0) (mirror y) (unit 1)
+  (symbol (lib_id "Switch:SW_Push") (at 250.19 102.87 0) (mirror y) (unit 1)
     (in_bom yes) (on_board yes) (dnp no)
-    (property "Reference" "SW53" (at 254 99.695 0)
+    (property "Reference" "SW53" (at 254 100.965 0)
       (effects (font (size 0.8 0.8)) (justify left))
     )
-    (property "Value" "SPACE" (at 250.19 101.6 0)
+    (property "Value" "SPACE" (at 250.19 102.87 0)
       (effects (font (size 0.6 0.6)))
     )
-    (property "Footprint" "Button_Switch_Keyboard:SW_Cherry_MX_1.00u_PCB" (at 250.19 96.52 0)
+    (property "Footprint" "RetroStackLibrary:SW_Cherry_MX_1.00u_PCB_Spacebar_Universal" (at 250.19 97.79 0)
       (effects (font (size 1.27 1.27)) hide)
     )
-    (property "Datasheet" "~" (at 250.19 96.52 0)
+    (property "Datasheet" "~" (at 250.19 97.79 0)
       (effects (font (size 1.27 1.27)) hide)
     )
